File: light_monitor.sch (KiCad schematic (older format))
At the start: 33 parts, among them IC1 TSL25911FN, J1 Conn_01x04_Male, J2 Conn_01x03_Male, J3 USB_B_Micro, U1 STM32L432KCUx, U2 STDC14, U3 TPS610986, U4 LDK130PU33R_DFN6, U5 RV-8803-C7, X1 board_lens

Commit message: R001 ordered from osh
Parts:
- IC1: symbol SamacSys_Parts:TSL25911FN -> light_monitor-rescue:TSL25911FN-SamacSys_Parts
- U3: symbol switch-mode-supply:TPS610986 -> light_monitor-rescue:TPS610986-switch-mode-supply
- U5: symbol bhimebau_rtc:RV-8803-C7 -> light_monitor-rescue:RV-8803-C7-bhimebau_rtc
- X1: symbol bhimebau-lens:board_lens -> light_monitor-rescue:board_lens-bhimebau-lens
Changed lines of the file:
@@
 	9750 6000 9500 6000
 $Comp
-L SamacSys_Parts:TSL25911FN IC1
+L light_monitor-rescue:TSL25911FN-SamacSys_Parts IC1
 U 1 1 5C6C255C
 P 8500 5900
@@
 $EndComp
 $Comp
-L switch-mode-supply:TPS610986 U3
+L light_monitor-rescue:TPS610986-switch-mode-supply U3
 U 1 1 5C6ED59E
 P 4450 4500
@@
 Connection ~ 4200 3500
 $Comp
-L bhimebau_rtc:RV-8803-C7 U5
+L light_monitor-rescue:RV-8803-C7-bhimebau_rtc U5
 U 1 1 5C73D671
 P 9000 4850
@@
 	1600 3100 1600 3250
 $Comp
-L bhimebau-lens:board_lens X1
+L light_monitor-rescue:board_lens-bhimebau-lens X1
 U 1 1 5C703045
 P 10350 6000

Commit message: added boot jumper
Parts:
- added J4: Conn_01x03_Male, Connector_PinHeader_2.54mm:PinHeader_1x03_P2.54mm_Vertical_SMD_Pin1Left, symbol Connector:Conn_01x03_Male
Connections:
- wire segments 127 -> 131
- no-connect marks 24 -> 23
Changed lines of the file:
@@
 NoConn ~ 8600 3000
 NoConn ~ 8600 2700
-NoConn ~ 8600 2400
 Text Label 8600 3100 2    50   ~ 0
 SWO
@@
 NoConn ~ 9600 2200
 NoConn ~ 9600 2300
+$Comp
+L Connector:Conn_01x03_Male J4
+U 1 1 5C784022
+P 7550 2400
+F 0 "J4" H 7656 2678 50  0000 C CNN
+F 1 "Conn_01x03_Male" H 7656 2587 50  0000 C CNN
+F 2 "Connector_PinHeader_2.54mm:PinHeader_1x03_P2.54mm_Vertical_SMD_Pin1Left" H 7550 2400 50  0001 C CNN
+F 3 "~" H 7550 2400 50  0001 C CNN
+	1    7550 2400
+	1    0    0    -1
+$EndComp
+Wire Wire Line
+	7750 2400 8600 2400
+$Comp
+L power:GND #PWR030
+U 1 1 5C7889D8
+P 7750 2600
+F 0 "#PWR030" H 7750 2350 50  0001 C CNN
+F 1 "GND" H 7755 2427 50  0000 C CNN
+F 2 "" H 7750 2600 50  0001 C CNN
+F 3 "" H 7750 2600 50  0001 C CNN
+	1    7750 2600
+	1    0    0    -1
+$EndComp
+$Comp
+L power:VDD #PWR031
+U 1 1 5C788A27
+P 8150 2250
+F 0 "#PWR031" H 8150 2100 50  0001 C CNN
+F 1 "VDD" H 8167 2423 50  0000 C CNN
+F 2 "" H 8150 2250 50  0001 C CNN
+F 3 "" H 8150 2250 50  0001 C CNN
+	1    8150 2250
+	1    0    0    -1
+$EndComp
+Wire Wire Line
+	7750 2300 8150 2300
+Wire Wire Line
+	8150 2300 8150 2250
+Wire Wire Line
+	7750 2500 7750 2600
 $EndSCHEMATC

Commit message: checkpoint
Parts:
- removed J4: Conn_01x03_Male, Connector_PinHeader_2.54mm:PinHeader_1x03_P2.54mm_Vertical_SMD_Pin1Left, symbol Connector:Conn_01x03_Male
Connections:
- wire segments 131 -> 127
- no-connect marks 23 -> 24
Changed lines of the file:
@@
 NoConn ~ 9600 2200
 NoConn ~ 9600 2300
-$Comp
-L Connector:Conn_01x03_Male J4
-U 1 1 5C784022
-P 7550 2400
-F 0 "J4" H 7656 2678 50  0000 C CNN
-F 1 "Conn_01x03_Male" H 7656 2587 50  0000 C CNN
-F 2 "Connector_PinHeader_2.54mm:PinHeader_1x03_P2.54mm_Vertical_SMD_Pin1Left" H 7550 2400 50  0001 C CNN
-F 3 "~" H 7550 2400 50  0001 C CNN
-	1    7550 2400
-	1    0    0    -1
-$EndComp
-Wire Wire Line
-	7750 2400 8600 2400
-$Comp
-L power:GND #PWR030
-U 1 1 5C7889D8
-P 7750 2600
-F 0 "#PWR030" H 7750 2350 50  0001 C CNN
-F 1 "GND" H 7755 2427 50  0000 C CNN
-F 2 "" H 7750 2600 50  0001 C CNN
-F 3 "" H 7750 2600 50  0001 C CNN
-	1    7750 2600
-	1    0    0    -1
-$EndComp
-$Comp
-L power:VDD #PWR031
-U 1 1 5C788A27
-P 8150 2250
-F 0 "#PWR031" H 8150 2100 50  0001 C CNN
-F 1 "VDD" H 8167 2423 50  0000 C CNN
-F 2 "" H 8150 2250 50  0001 C CNN
-F 3 "" H 8150 2250 50  0001 C CNN
-	1    8150 2250
-	1    0    0    -1
-$EndComp
-Wire Wire Line
-	7750 2300 8150 2300
-Wire Wire Line
-	8150 2300 8150 2250
-Wire Wire Line
-	7750 2500 7750 2600
+NoConn ~ 8600 2400
 $EndSCHEMATC

Commit message: beginning the process of cleaning up the pad issues
Parts:
- removed J1: Conn_01x04_Male, Connector_JST:JST_XH_B4B-XH-AM_1x04_P2.50mm_Vertical, symbol Connector:Conn_01x04_Male
- removed J2: Conn_01x03_Male, Connector_PinHeader_2.54mm:PinHeader_1x03_P2.54mm_Vertical_SMD_Pin1Left, symbol Connector:Conn_01x03_Male
- removed TP1: VOUT_MON, TestPoint:TestPoint_Pad_D1.0mm, symbol Connector:TestPoint
- added H1: MountingHole, MountingHole:MountingHole_2.2mm_M2, symbol Mechanical:MountingHole
- added JP1, JP2, JP3, JP4: Jumper_2_Open, Jumper:SolderJumper-2_P1.3mm_Open_RoundedPad1.0x1.5mm, symbol Jumper:Jumper_2_Open
- BT1: footprint Battery:BatteryHolder_Keystone_3034_1x20mm -> Battery:BatteryHolder_Keystone_1060_1x2032
- U3: footprint Package_SON:Texas_PWSON-N6 -> SON50P150X150X80-6N:SON50P150X150X80-6N
Connections:
- net labels added: VBATT
- wire segments 127 -> 124
- no-connect marks 24 -> 22
Other:
- note added: "Connect only one jumper pair!\nJP2/JP3 Connected: Boost Regulator\nJP1/JP4 Connected: Boost Regulator Bypassed"
- note removed: "Pwr Select Port"
- note removed: "ST Pwr Shield"
Changed lines of the file:
@@
 encoding utf-8
 Sheet 1 1
-Title "Light Sensor Prototype 1 "
+Title "Light Sensor Prototype "
 Date "2019-02-01"
-Rev "R001"
+Rev "R002"
 Comp "Indiana University"
 Comment1 "Bryce Himebaugh"
@@
 F 0 "BT1" H 2000 5050 50  0000 L CNN
 F 1 "Battery_Cell" H 2000 4950 50  0000 L CNN
-F 2 "Battery:BatteryHolder_Keystone_3034_1x20mm" V 2500 4860 50  0001 C CNN
+F 2 "Battery:BatteryHolder_Keystone_1060_1x2032" V 2500 4860 50  0001 C CNN
 F 3 "~" V 2500 4860 50  0001 C CNN
 	1    2500 4800
@@
 F 0 "U3" H 4450 4865 50  0000 C CNN
 F 1 "TPS610986" H 4450 4774 50  0000 C CNN
-F 2 "Package_SON:Texas_PWSON-N6" H 4450 4500 50  0001 C CNN
+F 2 "SON50P150X150X80-6N:SON50P150X150X80-6N" H 4450 4500 50  0001 C CNN
 F 3 "" H 4450 4500 50  0001 C CNN
 	1    4450 4500
-	1    0    0    -1
-$EndComp
-$Comp
-L Connector:Conn_01x04_Male J1
-U 1 1 5C6ED6FE
-P 2150 3600
-F 0 "J1" H 2256 3878 50  0000 C CNN
-F 1 "Conn_01x04_Male" H 2256 3787 50  0000 C CNN
-F 2 "Connector_JST:JST_XH_B4B-XH-AM_1x04_P2.50mm_Vertical" H 2150 3600 50  0001 C CNN
-F 3 "~" H 2150 3600 50  0001 C CNN
-	1    2150 3600
 	1    0    0    -1
 $EndComp
@@
 Wire Wire Line
 	4200 3300 4200 3500
-$Comp
-L Connector:Conn_01x03_Male J2
-U 1 1 5C715BF3
-P 2150 4150
-F 0 "J2" H 2256 4428 50  0000 C CNN
-F 1 "Conn_01x03_Male" H 2256 4337 50  0000 C CNN
-F 2 "Connector_PinHeader_2.54mm:PinHeader_1x03_P2.54mm_Vertical_SMD_Pin1Left" H 2150 4150 50  0001 C CNN
-F 3 "~" H 2150 4150 50  0001 C CNN
-	1    2150 4150
-	1    0    0    -1
-$EndComp
-Wire Wire Line
-	2500 4250 2350 4250
-Wire Wire Line
-	2500 4250 2500 4600
-Wire Wire Line
-	2350 4150 2900 4150
-Wire Wire Line
-	2900 4150 2900 4500
-Connection ~ 2900 4500
 Text Notes 2150 3200 0    50   ~ 0
 CN14
-$Comp
-L power:GND #PWR010
-U 1 1 5C71E489
-P 3000 3600
-F 0 "#PWR010" H 3000 3350 50  0001 C CNN
-F 1 "GND" H 3005 3427 50  0000 C CNN
-F 2 "" H 3000 3600 50  0001 C CNN
-F 3 "" H 3000 3600 50  0001 C CNN
-	1    3000 3600
-	1    0    0    -1
-$EndComp
-Wire Wire Line
-	2350 3500 3000 3500
-Wire Wire Line
-	3000 3500 3000 3600
-Wire Wire Line
-	2350 3700 2700 3700
-Wire Wire Line
-	2700 3700 2700 4050
-Wire Wire Line
-	2700 4050 2350 4050
-$Comp
-L Connector:TestPoint TP1
-U 1 1 5C72454F
-P 3000 4000
-F 0 "TP1" H 3058 4120 50  0000 L CNN
-F 1 "VOUT_MON" H 3058 4029 50  0000 L CNN
-F 2 "TestPoint:TestPoint_Pad_D1.0mm" H 3200 4000 50  0001 C CNN
-F 3 "~" H 3200 4000 50  0001 C CNN
-	1    3000 4000
-	1    0    0    -1
-$EndComp
-Wire Wire Line
-	2350 3800 2800 3800
-Wire Wire Line
-	2800 3800 2800 4050
-Wire Wire Line
-	2800 4050 3000 4050
-Wire Wire Line
-	3000 4050 3000 4000
 Connection ~ 4200 3500
 $Comp
@@
 NoConn ~ 9600 2800
 Wire Wire Line
-	3600 3500 3950 3500
-Wire Wire Line
-	3950 3500 3950 4400
-Connection ~ 3950 3500
-Wire Wire Line
-	3950 3500 4200 3500
-NoConn ~ 2350 3600
-Wire Wire Line
 	2500 4900 2500 5100
 NoConn ~ 3600 3750
@@
 	1    0    0    -1
 $EndComp
-Wire Wire Line
-	4200 3500 4550 3500
 Wire Wire Line
 	4800 2900 4800 3000
@@
 Wire Wire Line
 	6100 4100 6100 4300
-Wire Wire Line
-	6100 4300 5500 4300
-Connection ~ 5500 4300
-Text Notes 1450 4150 0    50   ~ 0
-Pwr Select Port
-Text Notes 1450 3700 0    50   ~ 0
-ST Pwr Shield
-$Comp
-L power:PWR_FLAG #FLG0101
-U 1 1 5C7B8AF0
-P 4550 3450
-F 0 "#FLG0101" H 4550 3525 50  0001 C CNN
-F 1 "PWR_FLAG" H 4550 3624 50  0000 C CNN
-F 2 "" H 4550 3450 50  0001 C CNN
-F 3 "~" H 4550 3450 50  0001 C CNN
-	1    4550 3450
-	1    0    0    -1
-$EndComp
-Wire Wire Line
-	4550 3450 4550 3500
-Connection ~ 4550 3500
-Wire Wire Line
-	4550 3500 5200 3500
 $Comp
 L power:PWR_FLAG #FLG0102
@@
 NoConn ~ 9600 2200
 NoConn ~ 9600 2300
-NoConn ~ 8600 2400
+Wire Wire Line
+	2500 4600 2500 4500
+Wire Wire Line
+	2500 4500 2900 4500
+Connection ~ 2900 4500
+$Comp
+L power:VDD #PWR0102
+U 1 1 5C7C8CE0
+P 7850 2250
+F 0 "#PWR0102" H 7850 2100 50  0001 C CNN
+F 1 "VDD" H 7867 2423 50  0000 C CNN
+F 2 "" H 7850 2250 50  0001 C CNN
+F 3 "" H 7850 2250 50  0001 C CNN
+	1    7850 2250
+	1    0    0    -1
+$EndComp
+Wire Wire Line
+	7850 2250 7850 2400
+Wire Wire Line
+	7850 2400 8600 2400
+$Comp
+L power:PWR_FLAG #FLG0101
+U 1 1 5C7CD34C
+P 1100 3050
+F 0 "#FLG0101" H 1100 3125 50  0001 C CNN
+F 1 "PWR_FLAG" H 1100 3224 50  0000 C CNN
+F 2 "" H 1100 3050 50  0001 C CNN
+F 3 "~" H 1100 3050 50  0001 C CNN
+	1    1100 3050
+	1    0    0    -1
+$EndComp
+Wire Wire Line
+	1100 3050 1100 3100
+Wire Wire Line
+	1100 3100 1500 3100
+Connection ~ 1500 3100
+Wire Wire Line
+	4200 3500 5200 3500
+$Comp
+L Jumper:Jumper_2_Open JP1
+U 1 1 5C85336F
+P 2500 3850
+F 0 "JP1" V 2454 3948 50  0000 L CNN
+F 1 "Jumper_2_Open" V 2545 3948 50  0000 L CNN
+F 2 "Jumper:SolderJumper-2_P1.3mm_Open_RoundedPad1.0x1.5mm" H 2500 3850 50  0001 C CNN
+F 3 "~" H 2500 3850 50  0001 C CNN
+	1    2500 3850
+	0    1    1    0
+$EndComp
+Wire Wire Line
+	2500 4050 2500 4500
+Connection ~ 2500 4500
+Wire Wire Line
+	2500 3650 2500 3500
+Wire Wire Line
+	2500 3500 3600 3500
+Connection ~ 3600 3500
+Text Label 2500 4500 0    50   ~ 0
+VBATT
+Wire Wire Line
+	3600 3500 3950 3500
+$Comp
+L Jumper:Jumper_2_Open JP2
+U 1 1 5C8601AA
+P 3950 3750
+F 0 "JP2" V 3904 3848 50  0000 L CNN
+F 1 "Jumper_2_Open" V 3995 3848 50  0000 L CNN
+F 2 "Jumper:SolderJumper-2_P1.3mm_Open_RoundedPad1.0x1.5mm" H 3950 3750 50  0001 C CNN
+F 3 "~" H 3950 3750 50  0001 C CNN
+	1    3950 3750
+	0    1    1    0
+$EndComp
+Wire Wire Line
+	3950 3550 3950 3500
+Connection ~ 3950 3500
+Wire Wire Line
+	3950 3500 4200 3500
+Wire Wire Line
+	3950 3950 3950 4400
+$Comp
+L Jumper:Jumper_2_Open JP3
+U 1 1 5C868F0D
+P 5750 4300
+F 0 "JP3" H 5750 4075 50  0000 C CNN
+F 1 "Jumper_2_Open" H 5750 4166 50  0000 C CNN
+F 2 "Jumper:SolderJumper-2_P1.3mm_Open_RoundedPad1.0x1.5mm" H 5750 4300 50  0001 C CNN
+F 3 "~" H 5750 4300 50  0001 C CNN
+	1    5750 4300
+	-1   0    0    1
+$EndComp
+Wire Wire Line
+	5500 4300 5550 4300
+Connection ~ 5500 4300
+Wire Wire Line
+	5950 4300 6100 4300
+$Comp
+L Jumper:Jumper_2_Open JP4
+U 1 1 5C871B08
+P 6450 4300
+F 0 "JP4" H 6450 4075 50  0000 C CNN
+F 1 "Jumper_2_Open" H 6450 4166 50  0000 C CNN
+F 2 "Jumper:SolderJumper-2_P1.3mm_Open_RoundedPad1.0x1.5mm" H 6450 4300 50  0001 C CNN
+F 3 "~" H 6450 4300 50  0001 C CNN
+	1    6450 4300
+	-1   0    0    1
+$EndComp
+Wire Wire Line
+	6100 4300 6250 4300
+Connection ~ 6100 4300
+Text Label 6650 4300 0    50   ~ 0
+VBATT
+Text Notes 600  4300 0    50   ~ 0
+Connect only one jumper pair!\nJP2/JP3 Connected: Boost Regulator\nJP1/JP4 Connected: Boost Regulator Bypassed
+$Comp
+L Mechanical:MountingHole H1
+U 1 1 5C876E19
+P 10350 5600
+F 0 "H1" H 10450 5646 50  0000 L CNN
+F 1 "MountingHole" H 10450 5555 50  0000 L CNN
+F 2 "MountingHole:MountingHole_2.2mm_M2" H 10350 5600 50  0001 C CNN
+F 3 "~" H 10350 5600 50  0001 C CNN
+	1    10350 5600
+	1    0    0    -1
+$EndComp
 $EndSCHEMATC

Commit message: sensor complete
Parts:
- removed C2, C5: 10uF, Capacitor_SMD:C_0603_1608Metric_Pad1.05x0.95mm_HandSolder, symbol Device:C
- removed C3: 0.1uF, Capacitor_SMD:C_0603_1608Metric_Pad1.05x0.95mm_HandSolder, symbol Device:C
- removed C4, C7: 1uF, Capacitor_SMD:C_0603_1608Metric_Pad1.05x0.95mm_HandSolder, symbol Device:C
- removed C6: 10nF, Capacitor_SMD:C_0603_1608Metric_Pad1.05x0.95mm_HandSolder, symbol Device:C
- removed D2, D3, D4, D5: D_Schottky, Diode_SMD:D_SOD-323, symbol Device:D_Schottky
- removed H1: MountingHole, MountingHole:MountingHole_2.2mm_M2, symbol Mechanical:MountingHole
- removed J3: USB_B_Micro, Connector_USB:USB_Micro-B_Molex_47346-0001, symbol Connector:USB_B_Micro
- removed JP1, JP2, JP3, JP4: Jumper_2_Open, Jumper:SolderJumper-2_P1.3mm_Open_RoundedPad1.0x1.5mm, symbol Jumper:Jumper_2_Open
- removed L1: 4.7uH, bhimebau_inductor:TDKVLF3025, symbol Device:L
- removed R3: 400, Resistor_SMD:R_0603_1608Metric_Pad1.05x0.95mm_HandSolder, symbol Device:R_US
- removed R4: 100k, Resistor_SMD:R_0603_1608Metric_Pad1.05x0.95mm_HandSolder, symbol Device:R_US
- removed U3: TPS610986, SON50P150X150X80-6N:SON50P150X150X80-6N, symbol light_monitor-rescue:TPS610986-switch-mode-supply
- removed U4: LDK130PU33R_DFN6, Package_DFN_QFN:DFN-6_1.3x1.2mm_P0.4mm, symbol Regulator_Linear:LDK130PU33R_DFN6
Connections:
- net labels added: rtc_EVI, rtc_nINT, sensor_int
- net labels removed: +3.3V, +VSW, SW_MODE, USB_N, USB_P, VBATT
- wire segments 124 -> 56
- no-connect marks 22 -> 18
Other:
- note added: "Pwr Select Port"
- note removed: "CN14"
- note removed: "Connect only one jumper pair!\nJP2/JP3 Connected: Boost Regulator\nJP1/JP4 Connected: Boost Regulator Bypassed"
- moved on the sheet: BT1, C1

Commit message: checking rev 4
Parts:
- added C2: 0.1uF, Capacitor_SMD:C_0603_1608Metric_Pad1.05x0.95mm_HandSolder, symbol Device:C
- BT1: footprint Battery:BatteryHolder_Keystone_1060_1x2032 -> bhimebau_battery:Keystone_1091TR
Connections:
- net GND: now also C2.2
- net VDD: no longer IC1.5 (VDD)
- net sensor_power: now reaches U1.21 (PA11)
- net sensor_power: now also IC1.5 (VDD), C2.1
- no-connect marks 18 -> 17
Changed lines of the file:
@@
 Title "Light Sensor Breakout "
 Date "2019-02-01"
-Rev "R003"
+Rev "R004"
 Comp "Indiana University"
 Comment1 "Bryce Himebaugh"
@@
 F 0 "BT1" H 4050 4000 50  0000 L CNN
 F 1 "Battery_Cell" H 4050 3900 50  0000 L CNN
-F 2 "Battery:BatteryHolder_Keystone_1060_1x2032" V 4550 3810 50  0001 C CNN
+F 2 "bhimebau_battery:Keystone_1091TR" V 4550 3810 50  0001 C CNN
 F 3 "~" V 4550 3810 50  0001 C CNN
 	1    4550 3750
@@
 Text Label 9500 6100 0    50   ~ 0
 sensor_data
-Wire Wire Line
-	9750 6000 9500 6000
 $Comp
 L light_monitor-rescue:TSL25911FN-SamacSys_Parts IC1
@@
 Wire Wire Line
 	5650 3100 5650 3000
-$Comp
-L power:VDD #PWR011
-U 1 1 5CDE1DE6
-P 9750 5700
-F 0 "#PWR011" H 9750 5550 50  0001 C CNN
-F 1 "VDD" H 9767 5873 50  0000 C CNN
-F 2 "" H 9750 5700 50  0001 C CNN
-F 3 "" H 9750 5700 50  0001 C CNN
-	1    9750 5700
-	1    0    0    -1
-$EndComp
-Wire Wire Line
-	9750 5700 9750 6000
 Wire Wire Line
 	8600 2400 7850 2400
@@
 Text Label 9600 2800 0    50   ~ 0
 sensor_int
-NoConn ~ 9600 3100
 NoConn ~ 9600 3200
 NoConn ~ 8600 3300
@@
 	4550 3100 4550 3550
 Connection ~ 4950 3100
+Text Label 9600 3100 0    50   ~ 0
+sensor_power
+Text Label 9500 6000 0    50   ~ 0
+sensor_power
+$Comp
+L Device:C C2
+U 1 1 5D1BBADB
+P 10400 4550
+F 0 "C2" H 10515 4596 50  0000 L CNN
+F 1 "0.1uF" H 10515 4505 50  0000 L CNN
+F 2 "Capacitor_SMD:C_0603_1608Metric_Pad1.05x0.95mm_HandSolder" H 10438 4400 50  0001 C CNN
+F 3 "~" H 10400 4550 50  0001 C CNN
+	1    10400 4550
+	1    0    0    -1
+$EndComp
+Text Label 10400 4200 0    50   ~ 0
+sensor_power
+$Comp
+L power:GND #PWR010
+U 1 1 5D1BC44D
+P 10400 5100
+F 0 "#PWR010" H 10400 4850 50  0001 C CNN
+F 1 "GND" H 10405 4927 50  0000 C CNN
+F 2 "" H 10400 5100 50  0001 C CNN
+F 3 "" H 10400 5100 50  0001 C CNN
+	1    10400 5100
+	1    0    0    -1
+$EndComp
+Wire Wire Line
+	10400 4700 10400 5100
+Wire Wire Line
+	10400 4400 10400 4200
 $EndSCHEMATC

Commit message: rev 005 lpuart sent to macrofab
Parts:
- removed X1: board_lens, bhimebau_inductor:carclo_lens, symbol light_monitor-rescue:board_lens-bhimebau-lens
- added J1: Conn_01x03, Connector_JST:JST_XH_B3B-XH-AM_1x03_P2.50mm_Vertical, symbol Connector_Generic:Conn_01x03
- added R3, R4: 200, Resistor_SMD:R_0603_1608Metric_Pad1.05x0.95mm_HandSolder, symbol Device:R_US
Connections:
- net GND: now also J1.3 (Pin_3)
- net RX: now also R4.1
- net TX: now also R3.1
- new net: J1.1 (Pin_1), R3.2
- new net: J1.2 (Pin_2), R4.2
Changed lines of the file:
@@
 Title "Light Sensor Breakout "
 Date "2019-02-01"
-Rev "R004"
+Rev "R005 lpuart"
 Comp "Indiana University"
 Comment1 "Bryce Himebaugh"
@@
 Pwr Select Port
 $Comp
-L light_monitor-rescue:board_lens-bhimebau-lens X1
-U 1 1 5C703045
-P 10350 6000
-F 0 "X1" H 10528 6046 50  0000 L CNN
-F 1 "board_lens" H 10528 5955 50  0000 L CNN
-F 2 "bhimebau_inductor:carclo_lens" H 10350 6000 50  0001 C CNN
-F 3 "" H 10350 6000 50  0001 C CNN
-	1    10350 6000
-	1    0    0    -1
-$EndComp
-$Comp
 L power:VDD #PWR022
 U 1 1 5C7046E7
@@
 Wire Wire Line
 	10400 4400 10400 4200
+$Comp
+L Device:R_US R3
+U 1 1 5D3772FC
+P 5000 4600
+F 0 "R3" V 4900 4550 50  0000 C CNN
+F 1 "200" V 4900 4700 50  0000 C CNN
+F 2 "Resistor_SMD:R_0603_1608Metric_Pad1.05x0.95mm_HandSolder" V 5040 4590 50  0001 C CNN
+F 3 "~" H 5000 4600 50  0001 C CNN
+	1    5000 4600
+	0    1    1    0
+$EndComp
+$Comp
+L Device:R_US R4
+U 1 1 5D3786E4
+P 5000 4700
+F 0 "R4" V 5100 4650 50  0000 C CNN
+F 1 "200" V 5100 4800 50  0000 C CNN
+F 2 "Resistor_SMD:R_0603_1608Metric_Pad1.05x0.95mm_HandSolder" V 5040 4690 50  0001 C CNN
+F 3 "~" H 5000 4700 50  0001 C CNN
+	1    5000 4700
+	0    1    1    0
+$EndComp
+Text Label 5150 4600 0    50   ~ 0
+TX
+Text Label 5150 4700 0    50   ~ 0
+RX
+$Comp
+L Connector_Generic:Conn_01x03 J1
+U 1 1 5D372F79
+P 4500 4700
+F 0 "J1" H 4418 5017 50  0000 C CNN
+F 1 "Conn_01x03" H 4418 4926 50  0000 C CNN
+F 2 "Connector_JST:JST_XH_B3B-XH-AM_1x03_P2.50mm_Vertical" H 4500 4700 50  0001 C CNN
+F 3 "~" H 4500 4700 50  0001 C CNN
+	1    4500 4700
+	-1   0    0    -1
+$EndComp
+Wire Wire Line
+	4700 4600 4850 4600
+Wire Wire Line
+	4700 4700 4850 4700
+$Comp
+L power:GND #PWR011
+U 1 1 5D38244E
+P 4900 4900
+F 0 "#PWR011" H 4900 4650 50  0001 C CNN
+F 1 "GND" H 4905 4727 50  0000 C CNN
+F 2 "" H 4900 4900 50  0001 C CNN
+F 3 "" H 4900 4900 50  0001 C CNN
+	1    4900 4900
+	1    0    0    -1
+$EndComp
+Wire Wire Line
+	4700 4800 4900 4800
+Wire Wire Line
+	4900 4800 4900 4900
 $EndSCHEMATC
