File: light_monitor.sch (KiCad schematic (older format))
At the start: 19 parts, among them IC1 TSL237S-LF, J1 Conn_01x03, J2 Conn_01x04_Male, U1 STM32L432KCUx, U2 STDC14, U3 TG-3541CE

Commit message: revision 8 sent to fab
Parts:
- removed C8: 2.2uF, Capacitor_SMD:C_0603_1608Metric_Pad1.05x0.95mm_HandSolder, symbol Device:C
- removed C9: 0.1uF, Capacitor_SMD:C_0603_1608Metric_Pad1.05x0.95mm_HandSolder, symbol Device:C
- removed JP2, JP3, JP4: Jumper_2_Open, Jumper:SolderJumper-2_P1.3mm_Open_RoundedPad1.0x1.5mm, symbol Jumper:Jumper_2_Open
- added H1, H2, H3, H4: MountingHole, MountingHole:MountingHole_2.2mm_M2_Pad_Via, symbol Mechanical:MountingHole
- added U4: sm_tsl237, bhimebau_lightsensor:tsl237t, symbol bhimebau_lightsensor:sm_tsl237
- BT1: footprint bhimebau_battery:Keystone_1091TR -> bhimebau_battery:BR2330A_Horizontal_Circular_Holes
- R1: value 300 -> 4.7k
Connections:
- net labels removed: l432_pwr
- wire segments 72 -> 71
Changed lines of the file:
@@
 EESchema Schematic File Version 4
-LIBS:light_monitor-cache
 EELAYER 30 0
 EELAYER END
@@
 F 0 "BT1" H 1800 4900 50  0000 L CNN
 F 1 "Battery_Cell" H 1800 4800 50  0000 L CNN
-F 2 "bhimebau_battery:Keystone_1091TR" V 2300 4710 50  0001 C CNN
+F 2 "bhimebau_battery:BR2330A_Horizontal_Circular_Holes" V 2300 4710 50  0001 C CNN
 F 3 "~" V 2300 4710 50  0001 C CNN
 	1    2300 4650
@@
 P 6600 4050
 F 0 "R1" H 6668 4096 50  0000 L CNN
-F 1 "300" H 6668 4005 50  0000 L CNN
+F 1 "4.7k" H 6668 4005 50  0000 L CNN
 F 2 "Resistor_SMD:R_0603_1608Metric_Pad1.05x0.95mm_HandSolder" V 6640 4040 50  0001 C CNN
 F 3 "~" H 6600 4050 50  0001 C CNN
@@
 Pwr Select Port
 $Comp
-L power:GND #PWR023
-U 1 1 5C70472C
-P 9100 3000
-F 0 "#PWR023" H 9100 2750 50  0001 C CNN
-F 1 "GND" H 9105 2827 50  0000 C CNN
-F 2 "" H 9100 3000 50  0001 C CNN
-F 3 "" H 9100 3000 50  0001 C CNN
-	1    9100 3000
-	1    0    0    -1
-$EndComp
-$Comp
-L Device:C C8
-U 1 1 5C70478F
-P 9100 2750
-F 0 "C8" H 9215 2796 50  0000 L CNN
-F 1 "2.2uF" H 9215 2705 50  0000 L CNN
-F 2 "Capacitor_SMD:C_0603_1608Metric_Pad1.05x0.95mm_HandSolder" H 9138 2600 50  0001 C CNN
-F 3 "~" H 9100 2750 50  0001 C CNN
-	1    9100 2750
-	1    0    0    -1
-$EndComp
-$Comp
-L Device:C C9
-U 1 1 5C70483B
-P 9550 2750
-F 0 "C9" H 9665 2796 50  0000 L CNN
-F 1 "0.1uF" H 9665 2705 50  0000 L CNN
-F 2 "Capacitor_SMD:C_0603_1608Metric_Pad1.05x0.95mm_HandSolder" H 9588 2600 50  0001 C CNN
-F 3 "~" H 9550 2750 50  0001 C CNN
-	1    9550 2750
-	1    0    0    -1
-$EndComp
-$Comp
-L power:GND #PWR025
-U 1 1 5C7048DE
-P 9550 3000
-F 0 "#PWR025" H 9550 2750 50  0001 C CNN
-F 1 "GND" H 9555 2827 50  0000 C CNN
-F 2 "" H 9550 3000 50  0001 C CNN
-F 3 "" H 9550 3000 50  0001 C CNN
-	1    9550 3000
-	1    0    0    -1
-$EndComp
-Wire Wire Line
-	9100 2550 9100 2600
-Wire Wire Line
-	9100 2900 9100 3000
-Wire Wire Line
-	9550 2550 9550 2600
-Wire Wire Line
-	9550 2900 9550 3000
-$Comp
 L Device:C C10
 U 1 1 5C71E025
@@
 Wire Wire Line
 	2300 2850 1700 2850
-Text Label 7900 2250 0    50   ~ 0
-l432_pwr
-Text Label 9100 1500 0    50   ~ 0
-l432_pwr
-Text Label 9550 1500 0    50   ~ 0
-l432_pwr
-Text Label 9100 2550 0    50   ~ 0
-l432_pwr
-Text Label 9550 2550 0    50   ~ 0
-l432_pwr
 $Comp
 L bhimebau-oscillator:TG-3541CE U3
@@
 $EndComp
 $Comp
-L Jumper:Jumper_2_Open JP2
-U 1 1 5D814EFD
-P 3600 3400
-F 0 "JP2" H 3600 3635 50  0000 C CNN
-F 1 "Jumper_2_Open" H 3600 3544 50  0000 C CNN
-F 2 "Jumper:SolderJumper-2_P1.3mm_Open_RoundedPad1.0x1.5mm" H 3600 3400 50  0001 C CNN
-F 3 "~" H 3600 3400 50  0001 C CNN
-	1    3600 3400
-	1    0    0    -1
-$EndComp
-$Comp
 L power:VDD #PWR09
 U 1 1 5D815950
@@
 	3200 3250 3200 3400
 Wire Wire Line
-	3200 3400 3400 3400
-Wire Wire Line
-	3800 3400 4150 3400
-Wire Wire Line
 	4150 3400 4150 3500
 Wire Wire Line
@@
 NoConn ~ 7400 3400
 NoConn ~ 7400 3900
-$Comp
-L Jumper:Jumper_2_Open JP3
-U 1 1 5D8324ED
-P 3850 2400
-F 0 "JP3" H 3850 2635 50  0000 C CNN
-F 1 "Jumper_2_Open" H 3850 2544 50  0000 C CNN
-F 2 "Jumper:SolderJumper-2_P1.3mm_Open_RoundedPad1.0x1.5mm" H 3850 2400 50  0001 C CNN
-F 3 "~" H 3850 2400 50  0001 C CNN
-	1    3850 2400
-	1    0    0    -1
-$EndComp
 $Comp
 L SamacSys_Parts:TSL237S-LF IC1
@@
 Wire Wire Line
 	4300 2300 4300 2650
-Wire Wire Line
-	4400 2400 4050 2400
 Text Label 3650 2400 2    50   ~ 0
 tsl237_pwr
-$Comp
-L Jumper:Jumper_2_Open JP4
-U 1 1 5D839505
-P 7200 2200
-F 0 "JP4" H 7200 2435 50  0000 C CNN
-F 1 "Jumper_2_Open" H 7200 2344 50  0000 C CNN
-F 2 "Jumper:SolderJumper-2_P1.3mm_Open_RoundedPad1.0x1.5mm" H 7200 2200 50  0001 C CNN
-F 3 "~" H 7200 2200 50  0001 C CNN
-	1    7200 2200
-	1    0    0    -1
-$EndComp
-Wire Wire Line
-	7400 2200 7900 2200
 Wire Wire Line
 	7900 2200 7900 2350
 Wire Wire Line
 	6800 2100 6800 2200
-Wire Wire Line
-	6800 2200 7000 2200
 $Comp
 L MCU_ST_STM32L4:STM32L432KCUx U1
@@
 Text Label 5400 2300 0    50   ~ 0
 tsl237_freq
+$Comp
+L bhimebau_lightsensor:sm_tsl237 U4
+U 1 1 5E2CA9E3
+P 4900 1350
+F 0 "U4" H 4900 1515 50  0000 C CNN
+F 1 "sm_tsl237" H 4900 1424 50  0000 C CNN
+F 2 "bhimebau_lightsensor:tsl237t" H 4900 1350 50  0001 C CNN
+F 3 "" H 4900 1350 50  0001 C CNN
+	1    4900 1350
+	1    0    0    -1
+$EndComp
+Text Label 5350 1450 0    50   ~ 0
+tsl237_freq
+$Comp
+L power:GND #PWR0101
+U 1 1 5E2CB871
+P 4350 1800
+F 0 "#PWR0101" H 4350 1550 50  0001 C CNN
+F 1 "GND" H 4355 1627 50  0000 C CNN
+F 2 "" H 4350 1800 50  0001 C CNN
+F 3 "" H 4350 1800 50  0001 C CNN
+	1    4350 1800
+	1    0    0    -1
+$EndComp
+Wire Wire Line
+	4350 1800 4350 1600
+Wire Wire Line
+	4350 1600 4450 1600
+Wire Wire Line
+	4450 1450 4350 1450
+Wire Wire Line
+	4350 1450 4350 1600
+Connection ~ 4350 1600
+Text Label 6300 1600 0    50   ~ 0
+tsl237_pwr
+Wire Wire Line
+	6800 2200 7900 2200
+$Comp
+L power:VDD #PWR013
+U 1 1 5E2F18A1
+P 9100 1500
+F 0 "#PWR013" H 9100 1350 50  0001 C CNN
+F 1 "VDD" H 9117 1673 50  0000 C CNN
+F 2 "" H 9100 1500 50  0001 C CNN
+F 3 "" H 9100 1500 50  0001 C CNN
+	1    9100 1500
+	1    0    0    -1
+$EndComp
+$Comp
+L power:VDD #PWR014
+U 1 1 5E2F1ED1
+P 9550 1500
+F 0 "#PWR014" H 9550 1350 50  0001 C CNN
+F 1 "VDD" H 9567 1673 50  0000 C CNN
+F 2 "" H 9550 1500 50  0001 C CNN
+F 3 "" H 9550 1500 50  0001 C CNN
+	1    9550 1500
+	1    0    0    -1
+$EndComp
+Wire Wire Line
+	3200 3400 4150 3400
+Wire Wire Line
+	3650 2400 4400 2400
+Wire Wire Line
+	5350 1600 6300 1600
+$Comp
+L Mechanical:MountingHole H1
+U 1 1 5E2FA5D5
+P 9500 4500
+F 0 "H1" H 9600 4546 50  0000 L CNN
+F 1 "MountingHole" H 9600 4455 50  0000 L CNN
+F 2 "MountingHole:MountingHole_2.2mm_M2_Pad_Via" H 9500 4500 50  0001 C CNN
+F 3 "~" H 9500 4500 50  0001 C CNN
+	1    9500 4500
+	1    0    0    -1
+$EndComp
+$Comp
+L Mechanical:MountingHole H2
+U 1 1 5E2FB10A
+P 10000 5000
+F 0 "H2" H 10100 5046 50  0000 L CNN
+F 1 "MountingHole" H 10100 4955 50  0000 L CNN
+F 2 "MountingHole:MountingHole_2.2mm_M2_Pad_Via" H 10000 5000 50  0001 C CNN
+F 3 "~" H 10000 5000 50  0001 C CNN
+	1    10000 5000
+	1    0    0    -1
+$EndComp
+$Comp
+L Mechanical:MountingHole H4
+U 1 1 5E2FB3A2
+P 9000 5000
+F 0 "H4" H 9100 5046 50  0000 L CNN
+F 1 "MountingHole" H 9100 4955 50  0000 L CNN
+F 2 "MountingHole:MountingHole_2.2mm_M2_Pad_Via" H 9000 5000 50  0001 C CNN
+F 3 "~" H 9000 5000 50  0001 C CNN
+	1    9000 5000
+	1    0    0    -1
+$EndComp
+$Comp
+L Mechanical:MountingHole H3
+U 1 1 5E2FB6E8
+P 9500 5500
+F 0 "H3" H 9600 5546 50  0000 L CNN
+F 1 "MountingHole" H 9600 5455 50  0000 L CNN
+F 2 "MountingHole:MountingHole_2.2mm_M2_Pad_Via" H 9500 5500 50  0001 C CNN
+F 3 "~" H 9500 5500 50  0001 C CNN
+	1    9500 5500
+	1    0    0    -1
+$EndComp
 $EndSCHEMATC

Commit message: sent to fab
Parts:
- added C1, C2: 2.2uF, Capacitor_SMD:C_0603_1608Metric_Pad1.05x0.95mm_HandSolder, symbol Device:C
- added C3: 0.1uF, Capacitor_SMD:C_0603_1608Metric_Pad1.05x0.95mm_HandSolder, symbol Device:C
- added R2: 1k, Resistor_SMD:R_0603_1608Metric_Pad1.05x0.95mm_HandSolder, symbol Device:R_US
- added U5: REG710-3, Package_TO_SOT_SMD:SOT-23-6_Handsoldering, symbol bhimebau-switch-mode-supply:REG710-3
Connections:
- net labels added: sensor_3v
- wire segments 71 -> 91
Changed lines of the file:
@@
 L power:GND #PWR010
 U 1 1 5D835550
-P 4300 2650
-F 0 "#PWR010" H 4300 2400 50  0001 C CNN
-F 1 "GND" H 4305 2477 50  0000 C CNN
-F 2 "" H 4300 2650 50  0001 C CNN
-F 3 "" H 4300 2650 50  0001 C CNN
-	1    4300 2650
-	1    0    0    -1
-$EndComp
-Wire Wire Line
-	4400 2300 4300 2300
-Wire Wire Line
-	4300 2300 4300 2650
-Text Label 3650 2400 2    50   ~ 0
-tsl237_pwr
+P 3900 2650
+F 0 "#PWR010" H 3900 2400 50  0001 C CNN
+F 1 "GND" H 3905 2477 50  0000 C CNN
+F 2 "" H 3900 2650 50  0001 C CNN
+F 3 "" H 3900 2650 50  0001 C CNN
+	1    3900 2650
+	1    0    0    -1
+$EndComp
 Wire Wire Line
 	7900 2200 7900 2350
@@
 NoConn ~ 1700 2750
 NoConn ~ 1700 2950
-Text Label 5400 2300 0    50   ~ 0
+Text Label 6600 1450 0    50   ~ 0
 tsl237_freq
 $Comp
@@
 	1    0    0    -1
 $EndComp
-Text Label 5350 1450 0    50   ~ 0
-tsl237_freq
 $Comp
 L power:GND #PWR0101
@@
 	4350 1450 4350 1600
 Connection ~ 4350 1600
-Text Label 6300 1600 0    50   ~ 0
-tsl237_pwr
 Wire Wire Line
 	6800 2200 7900 2200
@@
 Wire Wire Line
 	3200 3400 4150 3400
-Wire Wire Line
-	3650 2400 4400 2400
-Wire Wire Line
-	5350 1600 6300 1600
 $Comp
 L Mechanical:MountingHole H1
@@
 	1    0    0    -1
 $EndComp
+$Comp
+L bhimebau-switch-mode-supply:REG710-3 U5
+U 1 1 5E2D93B6
+P 2500 1550
+F 0 "U5" H 2525 1915 50  0000 C CNN
+F 1 "REG710-3" H 2525 1824 50  0000 C CNN
+F 2 "Package_TO_SOT_SMD:SOT-23-6_Handsoldering" H 2500 1550 50  0001 C CNN
+F 3 "" H 2500 1550 50  0001 C CNN
+	1    2500 1550
+	1    0    0    -1
+$EndComp
+$Comp
+L power:GND #PWR016
+U 1 1 5E2DAF04
+P 1400 1950
+F 0 "#PWR016" H 1400 1700 50  0001 C CNN
+F 1 "GND" H 1405 1777 50  0000 C CNN
+F 2 "" H 1400 1950 50  0001 C CNN
+F 3 "" H 1400 1950 50  0001 C CNN
+	1    1400 1950
+	1    0    0    -1
+$EndComp
+Wire Wire Line
+	1400 1950 1400 1550
+$Comp
+L power:VDD #PWR017
+U 1 1 5E2DCFA5
+P 3550 1500
+F 0 "#PWR017" H 3550 1350 50  0001 C CNN
+F 1 "VDD" H 3567 1673 50  0000 C CNN
+F 2 "" H 3550 1500 50  0001 C CNN
+F 3 "" H 3550 1500 50  0001 C CNN
+	1    3550 1500
+	1    0    0    -1
+$EndComp
+Wire Wire Line
+	3150 1550 3550 1550
+Wire Wire Line
+	3550 1550 3550 1500
+$Comp
+L Device:C C3
+U 1 1 5E2DFD30
+P 3900 1550
+F 0 "C3" H 4015 1596 50  0000 L CNN
+F 1 "0.1uF" H 4015 1505 50  0000 L CNN
+F 2 "Capacitor_SMD:C_0603_1608Metric_Pad1.05x0.95mm_HandSolder" H 3938 1400 50  0001 C CNN
+F 3 "~" H 3900 1550 50  0001 C CNN
+	1    3900 1550
+	1    0    0    -1
+$EndComp
+Wire Wire Line
+	3150 1450 3350 1450
+Wire Wire Line
+	3150 1650 3350 1650
+$Comp
+L Device:C C1
+U 1 1 5E2E4C94
+P 1050 1750
+F 0 "C1" H 1165 1796 50  0000 L CNN
+F 1 "2.2uF" H 1165 1705 50  0000 L CNN
+F 2 "Capacitor_SMD:C_0603_1608Metric_Pad1.05x0.95mm_HandSolder" H 1088 1600 50  0001 C CNN
+F 3 "~" H 1050 1750 50  0001 C CNN
+	1    1050 1750
+	1    0    0    -1
+$EndComp
+Wire Wire Line
+	1050 1600 1050 1450
+$Comp
+L power:GND #PWR015
+U 1 1 5E2E8431
+P 1050 1950
+F 0 "#PWR015" H 1050 1700 50  0001 C CNN
+F 1 "GND" H 1055 1777 50  0000 C CNN
+F 2 "" H 1050 1950 50  0001 C CNN
+F 3 "" H 1050 1950 50  0001 C CNN
+	1    1050 1950
+	1    0    0    -1
+$EndComp
+Wire Wire Line
+	1050 1900 1050 1950
+Wire Wire Line
+	1400 1550 1900 1550
+Wire Wire Line
+	1050 1450 1900 1450
+Text Label 1900 1650 2    50   ~ 0
+tsl237_pwr
+$Comp
+L Device:C C2
+U 1 1 5E2F7A01
+P 3550 1700
+F 0 "C2" H 3665 1746 50  0000 L CNN
+F 1 "2.2uF" H 3665 1655 50  0000 L CNN
+F 2 "Capacitor_SMD:C_0603_1608Metric_Pad1.05x0.95mm_HandSolder" H 3588 1550 50  0001 C CNN
+F 3 "~" H 3550 1700 50  0001 C CNN
+	1    3550 1700
+	1    0    0    -1
+$EndComp
+Connection ~ 3550 1550
+$Comp
+L power:GND #PWR018
+U 1 1 5E2F884D
+P 3550 1950
+F 0 "#PWR018" H 3550 1700 50  0001 C CNN
+F 1 "GND" H 3555 1777 50  0000 C CNN
+F 2 "" H 3550 1950 50  0001 C CNN
+F 3 "" H 3550 1950 50  0001 C CNN
+	1    3550 1950
+	1    0    0    -1
+$EndComp
+Wire Wire Line
+	3550 1850 3550 1950
+Wire Wire Line
+	3350 2200 3900 2200
+Wire Wire Line
+	3350 1650 3350 2200
+Wire Wire Line
+	3900 1700 3900 2200
+Wire Wire Line
+	3350 950  3900 950
+Wire Wire Line
+	3900 950  3900 1400
+Wire Wire Line
+	3350 950  3350 1450
+Text Label 950  1450 2    50   ~ 0
+sensor_3v
+Text Label 4400 2400 2    50   ~ 0
+sensor_3v
+Wire Wire Line
+	3900 2300 3900 2650
+Wire Wire Line
+	3900 2300 4400 2300
+Text Label 5350 1600 0    50   ~ 0
+sensor_3v
+$Comp
+L Device:R_US R2
+U 1 1 5E30948B
+P 6300 1450
+F 0 "R2" V 6200 1400 50  0000 C CNN
+F 1 "1k" V 6200 1550 50  0000 C CNN
+F 2 "Resistor_SMD:R_0603_1608Metric_Pad1.05x0.95mm_HandSolder" V 6340 1440 50  0001 C CNN
+F 3 "~" H 6300 1450 50  0001 C CNN
+	1    6300 1450
+	0    1    1    0
+$EndComp
+Wire Wire Line
+	5350 1450 5900 1450
+Wire Wire Line
+	5900 1450 5900 2300
+Wire Wire Line
+	5900 2300 5400 2300
+Connection ~ 5900 1450
+Wire Wire Line
+	5900 1450 6150 1450
+Wire Wire Line
+	6450 1450 6600 1450
+Wire Wire Line
+	950  1450 1050 1450
+Connection ~ 1050 1450
 $EndSCHEMATC

Commit message: saved off r009
Parts:
- removed D1: LED, LEDs:LED_0603_HandSoldering, symbol Device:LED
- removed R1: 4.7k, Resistor_SMD:R_0603_1608Metric_Pad1.05x0.95mm_HandSolder, symbol Device:R_US
- added D2: LED, LED_SMD:LED_0603_1608Metric_Pad1.05x0.95mm_HandSolder, symbol Device:LED
- added R5: 47k, Resistor_SMD:R_0603_1608Metric_Pad1.05x0.95mm_HandSolder, symbol Device:R_US
- added R6: 10k, Resistor_SMD:R_0603_1608Metric_Pad1.05x0.95mm_HandSolder, symbol Device:R_US
- added R7: 1k, Resistor_SMD:R_0603_1608Metric_Pad1.05x0.95mm_HandSolder, symbol Device:R_US
- added R8: 300, Resistor_SMD:R_0603_1608Metric_Pad1.05x0.95mm_HandSolder, symbol Device:R_US
- added U6: LT1677CS8, ltc1677:SO-8_S, symbol ltc1677:LT1677CS8
Connections:
- net labels added: current_feedback, dac_v, irange_0, irange_1, irange_2, irange_3
- wire segments 91 -> 100
- no-connect marks 24 -> 23
Other:
- moved on the sheet: C10, C11
Changed lines of the file:
@@
 Text Label 8400 4000 0    50   ~ 0
 SWDIO
-$Comp
-L Device:LED D1
-U 1 1 5C54B804
-P 6600 4450
-F 0 "D1" V 6638 4333 50  0000 R CNN
-F 1 "LED" V 6547 4333 50  0000 R CNN
-F 2 "LEDs:LED_0603_HandSoldering" H 6600 4450 50  0001 C CNN
-F 3 "~" H 6600 4450 50  0001 C CNN
-	1    6600 4450
-	0    -1   -1   0
-$EndComp
-$Comp
-L power:GND #PWR05
-U 1 1 5C54BF8A
-P 6600 4700
-F 0 "#PWR05" H 6600 4450 50  0001 C CNN
-F 1 "GND" H 6605 4527 50  0000 C CNN
-F 2 "" H 6600 4700 50  0001 C CNN
-F 3 "" H 6600 4700 50  0001 C CNN
-	1    6600 4700
-	1    0    0    -1
-$EndComp
-$Comp
-L Device:R_US R1
-U 1 1 5C54C3AB
-P 6600 4050
-F 0 "R1" H 6668 4096 50  0000 L CNN
-F 1 "4.7k" H 6668 4005 50  0000 L CNN
-F 2 "Resistor_SMD:R_0603_1608Metric_Pad1.05x0.95mm_HandSolder" V 6640 4040 50  0001 C CNN
-F 3 "~" H 6600 4050 50  0001 C CNN
-	1    6600 4050
-	1    0    0    -1
-$EndComp
-Wire Wire Line
-	6600 4200 6600 4300
-Wire Wire Line
-	6600 4600 6600 4700
 NoConn ~ 7400 3700
 Text Label 7400 3800 2    50   ~ 0
 SWO
-Wire Wire Line
-	6600 3600 7400 3600
-Wire Wire Line
-	6600 3600 6600 3900
 NoConn ~ 8400 4200
 Text Notes 3150 7400 0    50   ~ 0
@@
 L Device:C C10
 U 1 1 5C71E025
-P 9100 1750
-F 0 "C10" H 9215 1796 50  0000 L CNN
-F 1 "2.2uF" H 9215 1705 50  0000 L CNN
-F 2 "Capacitor_SMD:C_0603_1608Metric_Pad1.05x0.95mm_HandSolder" H 9138 1600 50  0001 C CNN
-F 3 "~" H 9100 1750 50  0001 C CNN
-	1    9100 1750
+P 10250 1700
+F 0 "C10" H 10365 1746 50  0000 L CNN
+F 1 "2.2uF" H 10365 1655 50  0000 L CNN
+F 2 "Capacitor_SMD:C_0603_1608Metric_Pad1.05x0.95mm_HandSolder" H 10288 1550 50  0001 C CNN
+F 3 "~" H 10250 1700 50  0001 C CNN
+	1    10250 1700
 	1    0    0    -1
 $EndComp
@@
 L Device:C C11
 U 1 1 5C71E089
-P 9550 1750
-F 0 "C11" H 9665 1796 50  0000 L CNN
-F 1 "0.1uF" H 9665 1705 50  0000 L CNN
-F 2 "Capacitor_SMD:C_0603_1608Metric_Pad1.05x0.95mm_HandSolder" H 9588 1600 50  0001 C CNN
-F 3 "~" H 9550 1750 50  0001 C CNN
-	1    9550 1750
+P 10750 1700
+F 0 "C11" H 10865 1746 50  0000 L CNN
+F 1 "0.1uF" H 10865 1655 50  0000 L CNN
+F 2 "Capacitor_SMD:C_0603_1608Metric_Pad1.05x0.95mm_HandSolder" H 10788 1550 50  0001 C CNN
+F 3 "~" H 10750 1700 50  0001 C CNN
+	1    10750 1700
 	1    0    0    -1
 $EndComp
@@
 L power:GND #PWR027
 U 1 1 5C71E18B
-P 9100 2050
-F 0 "#PWR027" H 9100 1800 50  0001 C CNN
-F 1 "GND" H 9105 1877 50  0000 C CNN
-F 2 "" H 9100 2050 50  0001 C CNN
-F 3 "" H 9100 2050 50  0001 C CNN
-	1    9100 2050
+P 10250 2000
+F 0 "#PWR027" H 10250 1750 50  0001 C CNN
+F 1 "GND" H 10255 1827 50  0000 C CNN
+F 2 "" H 10250 2000 50  0001 C CNN
+F 3 "" H 10250 2000 50  0001 C CNN
+	1    10250 2000
 	1    0    0    -1
 $EndComp
@@
 L power:GND #PWR029
 U 1 1 5C71E1D8
-P 9550 2050
-F 0 "#PWR029" H 9550 1800 50  0001 C CNN
-F 1 "GND" H 9555 1877 50  0000 C CNN
-F 2 "" H 9550 2050 50  0001 C CNN
-F 3 "" H 9550 2050 50  0001 C CNN
-	1    9550 2050
-	1    0    0    -1
-$EndComp
-Wire Wire Line
-	9100 1600 9100 1500
-Wire Wire Line
-	9550 1600 9550 1500
-Wire Wire Line
-	9100 1900 9100 2050
-Wire Wire Line
-	9550 1900 9550 2050
+P 10750 2000
+F 0 "#PWR029" H 10750 1750 50  0001 C CNN
+F 1 "GND" H 10755 1827 50  0000 C CNN
+F 2 "" H 10750 2000 50  0001 C CNN
+F 3 "" H 10750 2000 50  0001 C CNN
+	1    10750 2000
+	1    0    0    -1
+$EndComp
+Wire Wire Line
+	10250 1550 10250 1450
+Wire Wire Line
+	10750 1550 10750 1450
+Wire Wire Line
+	10250 1850 10250 2000
+Wire Wire Line
+	10750 1850 10750 2000
 $Comp
 L power:GND #PWR030
@@
 	6650 3100 6650 3300
 NoConn ~ 8400 3900
-NoConn ~ 7400 4000
 NoConn ~ 11400 5400
 Text Label 8400 2900 0    50   ~ 0
@@
 Text Label 8400 3000 0    50   ~ 0
 RX
-NoConn ~ 7400 4100
 $Comp
 L Device:R_US R3
@@
 Wire Wire Line
 	3700 5500 3700 5600
-Text Label 8400 3200 0    50   ~ 0
+Text Label 8400 2700 0    50   ~ 0
 tsl237_freq
 Text Label 8400 3100 0    50   ~ 0
 tsl237_pwr
-NoConn ~ 7400 4200
 Wire Wire Line
 	6000 2700 7400 2700
@@
 	5600 3600 5600 3950
 NoConn ~ 7400 3400
-NoConn ~ 7400 3900
 $Comp
 L SamacSys_Parts:TSL237S-LF IC1
@@
 	1    0    0    -1
 $EndComp
-NoConn ~ 8400 2700
 NoConn ~ 8400 2800
 NoConn ~ 8400 3300
@@
 L power:VDD #PWR013
 U 1 1 5E2F18A1
-P 9100 1500
-F 0 "#PWR013" H 9100 1350 50  0001 C CNN
-F 1 "VDD" H 9117 1673 50  0000 C CNN
-F 2 "" H 9100 1500 50  0001 C CNN
-F 3 "" H 9100 1500 50  0001 C CNN
-	1    9100 1500
+P 10250 1450
+F 0 "#PWR013" H 10250 1300 50  0001 C CNN
+F 1 "VDD" H 10267 1623 50  0000 C CNN
+F 2 "" H 10250 1450 50  0001 C CNN
+F 3 "" H 10250 1450 50  0001 C CNN
+	1    10250 1450
 	1    0    0    -1
 $EndComp
@@
 L power:VDD #PWR014
 U 1 1 5E2F1ED1
-P 9550 1500
-F 0 "#PWR014" H 9550 1350 50  0001 C CNN
-F 1 "VDD" H 9567 1673 50  0000 C CNN
-F 2 "" H 9550 1500 50  0001 C CNN
-F 3 "" H 9550 1500 50  0001 C CNN
-	1    9550 1500
+P 10750 1450
+F 0 "#PWR014" H 10750 1300 50  0001 C CNN
+F 1 "VDD" H 10767 1623 50  0000 C CNN
+F 2 "" H 10750 1450 50  0001 C CNN
+F 3 "" H 10750 1450 50  0001 C CNN
+	1    10750 1450
 	1    0    0    -1
 $EndComp
@@
 	950  1450 1050 1450
 Connection ~ 1050 1450
+$Comp
+L ltc1677:LT1677CS8 U6
+U 1 1 5E3DB9E3
+P 7350 1150
+F 0 "U6" H 8350 1515 50  0000 C CNN
+F 1 "LT1677CS8" H 8350 1424 50  0000 C CNN
+F 2 "ltc1677:SO-8_S" H 7350 1150 50  0001 L BNN
+F 3 "lt1677cs8" H 7350 1150 50  0001 L BNN
+F 4 "Linear Technology" H 7350 1150 50  0001 L BNN "Field4"
+	1    7350 1150
+	1    0    0    -1
+$EndComp
+$Comp
+L power:GND #PWR019
+U 1 1 5E3E0C83
+P 7150 1550
+F 0 "#PWR019" H 7150 1300 50  0001 C CNN
+F 1 "GND" H 7155 1377 50  0000 C CNN
+F 2 "" H 7150 1550 50  0001 C CNN
+F 3 "" H 7150 1550 50  0001 C CNN
+	1    7150 1550
+	1    0    0    -1
+$EndComp
+Wire Wire Line
+	7350 1450 7150 1450
+Wire Wire Line
+	7150 1450 7150 1550
+Text Label 9350 1250 0    50   ~ 0
+sensor_3v
+$Comp
+L Device:LED D2
+U 1 1 5E3F7C7B
+P 9650 1850
+F 0 "D2" V 9688 1733 50  0000 R CNN
+F 1 "LED" V 9597 1733 50  0000 R CNN
+F 2 "LED_SMD:LED_0603_1608Metric_Pad1.05x0.95mm_HandSolder" H 9650 1850 50  0001 C CNN
+F 3 "~" H 9650 1850 50  0001 C CNN
+	1    9650 1850
+	0    -1   -1   0
+$EndComp
+Wire Wire Line
+	9350 1350 9650 1350
+Wire Wire Line
+	9650 1350 9650 1700
+$Comp
+L Device:R_US R7
+U 1 1 5E3FBDD0
+P 9650 2450
+F 0 "R7" H 9718 2496 50  0000 L CNN
+F 1 "1k" H 9718 2405 50  0000 L CNN
+F 2 "Resistor_SMD:R_0603_1608Metric_Pad1.05x0.95mm_HandSolder" V 9690 2440 50  0001 C CNN
+F 3 "~" H 9650 2450 50  0001 C CNN
+	1    9650 2450
+	1    0    0    -1
+$EndComp
+$Comp
+L Device:R_US R6
+U 1 1 5E3FC710
+P 9350 2450
+F 0 "R6" H 9418 2496 50  0000 L CNN
+F 1 "10k" H 9418 2405 50  0000 L CNN
+F 2 "Resistor_SMD:R_0603_1608Metric_Pad1.05x0.95mm_HandSolder" V 9390 2440 50  0001 C CNN
+F 3 "~" H 9350 2450 50  0001 C CNN
+	1    9350 2450
+	1    0    0    -1
+$EndComp
+$Comp
+L Device:R_US R5
+U 1 1 5E3FCA15
+P 9050 2450
+F 0 "R5" H 9118 2496 50  0000 L CNN
+F 1 "47k" H 9118 2405 50  0000 L CNN
+F 2 "Resistor_SMD:R_0603_1608Metric_Pad1.05x0.95mm_HandSolder" V 9090 2440 50  0001 C CNN
+F 3 "~" H 9050 2450 50  0001 C CNN
+	1    9050 2450
+	1    0    0    -1
+$EndComp
+$Comp
+L Device:R_US R8
+U 1 1 5E3FCD84
+P 9950 2450
+F 0 "R8" H 10018 2496 50  0000 L CNN
+F 1 "300" H 10018 2405 50  0000 L CNN
+F 2 "Resistor_SMD:R_0603_1608Metric_Pad1.05x0.95mm_HandSolder" V 9990 2440 50  0001 C CNN
+F 3 "~" H 9950 2450 50  0001 C CNN
+	1    9950 2450
+	1    0    0    -1
+$EndComp
+Wire Wire Line
+	9650 2000 9650 2150
+Wire Wire Line
+	9050 2150 9050 2300
+Connection ~ 9650 2150
+Wire Wire Line
+	9650 2150 9650 2300
+Wire Wire Line
+	9350 2300 9350 2150
+Connection ~ 9350 2150
+Wire Wire Line
+	9350 2150 9650 2150
+Wire Wire Line
+	9650 2150 9950 2150
+Wire Wire Line
+	9950 2150 9950 2300
+Text Label 7350 1250 2    50   ~ 0
+current_feedback
+Wire Wire Line
+	9050 2150 9350 2150
+Wire Wire Line
+	8800 2150 9050 2150
+Connection ~ 9050 2150
+Text Label 8800 2150 2    50   ~ 0
+current_feedback
+Text Label 7350 1350 2    50   ~ 0
+dac_v
+Text Label 8400 3200 0    50   ~ 0
+dac_v
+Text Label 9950 2600 3    50   ~ 0
+irange_0
+Text Label 9650 2600 3    50   ~ 0
+irange_1
+Text Label 9350 2600 3    50   ~ 0
+irange_2
+Text Label 9050 2600 3    50   ~ 0
+irange_3
+Text Label 7400 3900 2    50   ~ 0
+irange_0
+Text Label 7400 4000 2    50   ~ 0
+irange_1
+Text Label 7400 4100 2    50   ~ 0
+irange_2
+Text Label 7400 4200 2    50   ~ 0
+irange_3
+NoConn ~ 9350 1150
+NoConn ~ 9350 1450
+NoConn ~ 7350 1150
+NoConn ~ 7400 3600
 $EndSCHEMATC
