File: light_monitor.sch (KiCad schematic (older format))
At the start: 47 parts, among them IC1 TSL237S-LF, J1 Conn_01x03, J2 Conn_01x04_Male, U1 STM32L432KCUx, U2 STDC14, U3 TG-3541CE, U4 TPS7A05, U5 TPS22917, U6 AD8515

Commit message: board with lipo battery
Parts:
- R1, R9: renamed from 1k; value R_US -> 10k
- R8: value 300 -> 316
Changed lines of the file:
@@
 P 9950 2450
 F 0 "R8" H 10018 2496 50  0000 L CNN
-F 1 "300" H 10018 2405 50  0000 L CNN
+F 1 "316" H 10018 2405 50  0000 L CNN
 F 2 "Resistor_SMD:R_0603_1608Metric_Pad1.05x0.95mm_HandSolder" V 9990 2440 50  0001 C CNN
 F 3 "~" H 9950 2450 50  0001 C CNN
@@
 	9000 850  9000 1000
 $Comp
-L Device:R_US 1k
+L Device:R_US R9
 U 1 1 5E5FC201
 P 4750 2150
-F 0 "1k" H 4818 2196 50  0000 L CNN
-F 1 "R_US" H 4818 2105 50  0000 L CNN
+F 0 "R9" H 4818 2196 50  0000 L CNN
+F 1 "10k" H 4818 2105 50  0000 L CNN
 F 2 "Resistor_SMD:R_0603_1608Metric_Pad1.05x0.95mm_HandSolder" V 4790 2140 50  0001 C CNN
 F 3 "~" H 4750 2150 50  0001 C CNN
@@
 	4750 1850 4750 2000
 $Comp
-L Device:R_US 1k
+L Device:R_US R1
 U 1 1 5E600377
 P 4750 2550
-F 0 "1k" H 4818 2596 50  0000 L CNN
-F 1 "R_US" H 4818 2505 50  0000 L CNN
+F 0 "R1" H 4818 2596 50  0000 L CNN
+F 1 "10k" H 4818 2505 50  0000 L CNN
 F 2 "Resistor_SMD:R_0603_1608Metric_Pad1.05x0.95mm_HandSolder" V 4790 2540 50  0001 C CNN
 F 3 "~" H 4750 2550 50  0001 C CNN

Commit message: save off before access from freecad
Parts:
- added D1: LED, LED_SMD:LED_0603_1608Metric_Pad1.05x0.95mm_HandSolder, symbol Device:LED
- added R13: 4.7k, Resistor_SMD:R_0603_1608Metric_Pad1.05x0.95mm_HandSolder, symbol Device:R_US
- R11, R12: value R_US -> 100k
Connections:
- net GND: now also D1.1 (K)
- net at U1.14 (PB0): now also R13.1
- new net: D1.2 (A), R13.2
- no-connect marks 18 -> 17
Changed lines of the file:
@@
 Text Label 7400 4200 2    50   ~ 0
 irange_3
-NoConn ~ 7400 3600
 $Comp
 L Device:C C4
@@
 P 7850 1250
 F 0 "R11" V 7645 1250 50  0000 C CNN
-F 1 "R_US" V 7736 1250 50  0000 C CNN
+F 1 "100k" V 7736 1250 50  0000 C CNN
 F 2 "Resistor_SMD:R_0603_1608Metric_Pad1.05x0.95mm_HandSolder" V 7890 1240 50  0001 C CNN
 F 3 "~" H 7850 1250 50  0001 C CNN
@@
 P 8050 1450
 F 0 "R12" H 8118 1496 50  0000 L CNN
-F 1 "R_US" H 8118 1405 50  0000 L CNN
+F 1 "100k" H 8118 1405 50  0000 L CNN
 F 2 "Resistor_SMD:R_0603_1608Metric_Pad1.05x0.95mm_HandSolder" V 8090 1440 50  0001 C CNN
 F 3 "~" H 8050 1450 50  0001 C CNN
@@
 	1    0    0    -1
 $EndComp
+$Comp
+L Device:R_US R13
+U 1 1 5EC48AD7
+P 6450 3850
+F 0 "R13" H 6518 3896 50  0000 L CNN
+F 1 "4.7k" H 6518 3805 50  0000 L CNN
+F 2 "Resistor_SMD:R_0603_1608Metric_Pad1.05x0.95mm_HandSolder" V 6490 3840 50  0001 C CNN
+F 3 "~" H 6450 3850 50  0001 C CNN
+	1    6450 3850
+	1    0    0    -1
+$EndComp
+$Comp
+L Device:LED D1
+U 1 1 5EC4A020
+P 6450 4300
+F 0 "D1" V 6488 4183 50  0000 R CNN
+F 1 "LED" V 6397 4183 50  0000 R CNN
+F 2 "LED_SMD:LED_0603_1608Metric_Pad1.05x0.95mm_HandSolder" H 6450 4300 50  0001 C CNN
+F 3 "~" H 6450 4300 50  0001 C CNN
+	1    6450 4300
+	0    -1   -1   0
+$EndComp
+Wire Wire Line
+	7400 3600 6450 3600
+Wire Wire Line
+	6450 3600 6450 3700
+Wire Wire Line
+	6450 4000 6450 4150
+$Comp
+L power:GND #PWR038
+U 1 1 5EC58391
+P 6450 4700
+F 0 "#PWR038" H 6450 4450 50  0001 C CNN
+F 1 "GND" H 6455 4527 50  0000 C CNN
+F 2 "" H 6450 4700 50  0001 C CNN
+F 3 "" H 6450 4700 50  0001 C CNN
+	1    6450 4700
+	1    0    0    -1
+$EndComp
+Wire Wire Line
+	6450 4450 6450 4700
 $EndSCHEMATC

Commit message: added all changed files
Parts:
- J1: footprint Connector_JST:JST_XH_B3B-XH-AM_1x03_P2.50mm_Vertical -> Connector_JST:JST_XH_B3B-XH-A_1x03_P2.50mm_Vertical
- J2: footprint Connector_JST:JST_XH_B4B-XH-AM_1x04_P2.50mm_Vertical -> Connector_JST:JST_XH_B4B-XH-A_1x04_P2.50mm_Vertical
- U1: footprint Housings_DFN_QFN:QFN-32-1EP_5x5mm_Pitch0.5mm -> Package_DFN_QFN:QFN-32-1EP_5x5mm_P0.5mm_EP3.6x3.6mm
Changed lines of the file:
@@
 F 0 "J1" H 3218 5717 50  0000 C CNN
 F 1 "Conn_01x03" H 3218 5626 50  0000 C CNN
-F 2 "Connector_JST:JST_XH_B3B-XH-AM_1x03_P2.50mm_Vertical" H 3300 5400 50  0001 C CNN
+F 2 "Connector_JST:JST_XH_B3B-XH-A_1x03_P2.50mm_Vertical" H 3300 5400 50  0001 C CNN
 F 3 "~" H 3300 5400 50  0001 C CNN
 	1    3300 5400
@@
 F 0 "J2" H 1608 3131 50  0000 C CNN
 F 1 "Conn_01x04_Male" H 1608 3040 50  0000 C CNN
-F 2 "Connector_JST:JST_XH_B4B-XH-AM_1x04_P2.50mm_Vertical" H 1500 2850 50  0001 C CNN
+F 2 "Connector_JST:JST_XH_B4B-XH-A_1x04_P2.50mm_Vertical" H 1500 2850 50  0001 C CNN
 F 3 "~" H 1500 2850 50  0001 C CNN
 	1    1500 2850
@@
 F 0 "U1" H 8080 4320 50  0000 C CNN
 F 1 "STM32L432KCUx" H 8350 4250 50  0000 C CNN
-F 2 "Housings_DFN_QFN:QFN-32-1EP_5x5mm_Pitch0.5mm" H 7500 2500 50  0001 R CNN
+F 2 "Package_DFN_QFN:QFN-32-1EP_5x5mm_P0.5mm_EP3.6x3.6mm" H 7500 2500 50  0001 R CNN
 F 3 "http://www.st.com/st-web-ui/static/active/en/resource/technical/document/datasheet/DM00257205.pdf" H 7900 3400 50  0001 C CNN
 	1    7900 3400
