File: light_monitor.kicad_pcb (KiCad board)
At the start: 2 copper layers, 50.2 x 50.2 mm, 21 parts, among them IC1 TSL237S-LF, J1 Conn_01x03, J2 Conn_01x04_Male, U1 STM32L432KCUx, U2 STDC14, U3 TG-3541CE

Commit message: revision 8 sent to fab
Parts:
- removed C8: 2.2uF, Capacitor_SMD:C_0603_1608Metric_Pad1.05x0.95mm_HandSolder
- removed C9: 0.1uF, Capacitor_SMD:C_0603_1608Metric_Pad1.05x0.95mm_HandSolder
- removed IC1: TSL237S-LF, SamacSys_Parts_3:TSL237S-LF
- removed JP2, JP3, JP4: Jumper_2_Open, Jumper:SolderJumper-2_P1.3mm_Open_RoundedPad1.0x1.5mm
- added H1: MountingHole, MountingHole:MountingHole_2.2mm_M2_Pad_Via, F.Cu at (113.5, 83.5)
- added H2: MountingHole, MountingHole:MountingHole_2.2mm_M2_Pad_Via, F.Cu at (135.0, 105.0)
- added H3: MountingHole, MountingHole:MountingHole_2.2mm_M2_Pad_Via, F.Cu at (113.5, 126.5)
- added H4: MountingHole, MountingHole:MountingHole_2.2mm_M2_Pad_Via, F.Cu at (92.0, 105.0)
- added U4: sm_tsl237, bhimebau_lightsensor:tsl237t, F.Cu at (114.1, 102.2)
- added e: TSL237S-LF, SamacSys_Parts_3:TSL237S-LF, F.Cu at (113.5, 90.4)
- BT1: footprint bhimebau_battery:Keystone_1091TR -> bhimebau_battery:BR2330A_Horizontal_Circular_Holes
- C10, C11, JP1: moved to F.Cu
- R1: value 300 -> 4.7k; moved to F.Cu
- moved U2 34.8 mm to (97.9, 94.5)
- moved R3 31.0 mm to (103.0, 123.7), turned to 0 degrees
- moved R4 29.8 mm to (103.0, 125.5), turned to 0 degrees
- moved D1 19.8 mm to (109.0, 104.7), turned to 90 degrees
- moved R1 18.6 mm to (105.0, 102.1), turned to 0 degrees
- moved J2 15.8 mm to (124.2, 88.6), turned to 315 degrees
- moved JP1 14.7 mm to (125.8, 98.0)
- moved G*** 11.1 mm to (107.5, 114.2)
- moved G*** 10.3 mm to (119.0, 114.0)
- moved C10 9.96 mm to (97.4, 112.8), turned to 0 degrees
- moved C11 7.50 mm to (97.4, 111.1), turned to 0 degrees
- moved BT1 2.96 mm to (115.5, 105.3), turned to 90 degrees
- moved U1 1.13 mm to (97.4, 112.0)
- moved U3 1.13 mm to (94.6, 119.3)
Connections:
- C10 pad 1: /l432_pwr -> VDD
- C11 pad 1: /l432_pwr -> VDD
- U1 pad 1: /l432_pwr -> VDD
- U1 pad 17: /l432_pwr -> VDD
- U1 pad 5: /l432_pwr -> VDD
- U3 pad 1: Net-(JP2-Pad2) -> VDD
- U3 pad 2: Net-(JP2-Pad2) -> VDD
- U3 pad 3: Net-(JP2-Pad2) -> VDD
Routing:
- net /l432_pwr: track 38.3 -> 0.00 mm, vias 5 -> 0
- net Net-(R1-Pad1): track 54.3 -> 18.9 mm, vias 6 -> 3
- net /SWDCLK: track 36.0 -> 15.5 mm, vias 4 -> 2
- net /SWDIO: track 34.7 -> 15.0 mm, vias 4 -> 1
- net /TX: track 64.4 -> 46.4 mm, vias 3 -> 4
- net Net-(J1-Pad1): track 7.70 -> 25.5 mm, vias 1 -> 0
- net /NRST: track 42.1 -> 24.6 mm, vias 6 -> 2
- net Net-(J1-Pad2): track 9.22 -> 23.3 mm
- net /SWO: track 30.3 -> 18.0 mm, vias 4 -> 2
- net Net-(JP2-Pad2): track 11.7 -> 0.00 mm, vias 2 -> 0
- net Net-(BT1-Pad1): track 16.5 -> 6.00 mm
- net /tsl237_pwr: track 35.8 -> 46.3 mm, vias 4 -> 1
- net Net-(IC1-Pad2): track 9.63 -> 0.00 mm
- net VDD: track 22.6 -> 15.7 mm, vias 5 -> 4
- net Net-(J2-Pad2): track 9.22 -> 6.38 mm
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Other:
- board size 50.2 x 50.2 mm -> 50 x 50 mm
- board text added: "Dark Sky Detector R008"
- board text removed: "Light Monitor R007 Contact Information: Bryce Himebaugh bhimebau@indiana.edu 812-325-6673"
- board text removed: "batt"
- board text removed: "board"
- board text removed: "mon"

Commit message: sent to fab
Parts:
- added C1: 2.2uF, Capacitor_SMD:C_0603_1608Metric_Pad1.05x0.95mm_HandSolder, F.Cu at (107.0, 87.0)
- added C2: 2.2uF, Capacitor_SMD:C_0603_1608Metric_Pad1.05x0.95mm_HandSolder, F.Cu at (104.1, 87.0)
- added C3: 0.1uF, Capacitor_SMD:C_0603_1608Metric_Pad1.05x0.95mm_HandSolder, B.Cu at (102.0, 87.0)
- added R2: 1k, Resistor_SMD:R_0603_1608Metric_Pad1.05x0.95mm_HandSolder, F.Cu at (105.2, 108.6)
- added U5: REG710-3, Package_TO_SOT_SMD:SOT-23-6_Handsoldering, B.Cu at (105.5, 87.0)
- renumbered e to IC1
Connections:
- IC1 pad 2: /tsl237_pwr -> /sensor_3v
- IC1 pad 3: /tsl237_freq -> Net-(IC1-Pad3)
- J2 pad 1: (no net) -> Net-(J2-Pad1)
- J2 pad 3: (no net) -> Net-(J2-Pad3)
- U1 pad 12: (no net) -> Net-(U1-Pad12)
- U1 pad 13: (no net) -> Net-(U1-Pad13)
- U1 pad 15: (no net) -> Net-(U1-Pad15)
- U1 pad 18: (no net) -> Net-(U1-Pad18)
- U1 pad 19: (no net) -> Net-(U1-Pad19)
- U1 pad 20: (no net) -> Net-(U1-Pad20)
- U1 pad 21: (no net) -> Net-(U1-Pad21)
- U1 pad 22: (no net) -> Net-(U1-Pad22)
- U1 pad 25: (no net) -> Net-(U1-Pad25)
- U1 pad 27: (no net) -> Net-(U1-Pad27)
- U1 pad 28: (no net) -> Net-(U1-Pad28)
- U1 pad 29: (no net) -> Net-(U1-Pad29)
- U1 pad 3: (no net) -> Net-(U1-Pad3)
- U1 pad 30: (no net) -> Net-(U1-Pad30)
- U1 pad 6: (no net) -> Net-(U1-Pad6)
- U1 pad 7: (no net) -> Net-(U1-Pad7)
- U2 pad 1: (no net) -> Net-(U2-Pad1)
- U2 pad 10: (no net) -> Net-(U2-Pad10)
- U2 pad 2: (no net) -> Net-(U2-Pad2)
- U2 pad 9: (no net) -> Net-(U2-Pad9)
- U3 pad 10: (no net) -> Net-(U3-Pad10)
- U3 pad 6: (no net) -> Net-(U3-Pad6)
- U4 pad 3: /tsl237_pwr -> /sensor_3v
- U4 pad 4: /tsl237_freq -> Net-(IC1-Pad3)
Routing:
- net /sensor_3v: track 0.00 -> 29.0 mm, vias 0 -> 1
- net /tsl237_freq: track 43.8 -> 17.3 mm
- net Net-(IC1-Pad3): track 0.00 -> 26.0 mm
- net /tsl237_pwr: track 46.3 -> 35.2 mm, vias 1 -> 4
- net GND: track 45.3 -> 51.3 mm, vias 6 -> 7
- net VDD: track 15.7 -> 18.8 mm, vias 4 -> 5
- net Net-(C3-Pad2): track 0.00 -> 2.18 mm
- net Net-(C3-Pad1): track 0.00 -> 2.18 mm
- net /SWDIO: track 15.0 -> 15.7 mm, vias 1 -> 2

Commit message: saved off r009
Parts:
- removed D1: LED, LEDs:LED_0603_HandSoldering
- removed G***: LOGO, logo:iu_trident
- removed G***: LOGO, logo:hnf_logo
- removed R1: 4.7k, Resistor_SMD:R_0603_1608Metric_Pad1.05x0.95mm_HandSolder
- added D2: LED, LED_SMD:LED_0603_1608Metric_Pad1.05x0.95mm_HandSolder, F.Cu at (108.8, 104.9)
- added R5: 47k, Resistor_SMD:R_0603_1608Metric_Pad1.05x0.95mm_HandSolder, F.Cu at (109.0, 94.9)
- added R6: 10k, Resistor_SMD:R_0603_1608Metric_Pad1.05x0.95mm_HandSolder, F.Cu at (107.4, 94.9)
- added R7: 1k, Resistor_SMD:R_0603_1608Metric_Pad1.05x0.95mm_HandSolder, F.Cu at (105.8, 94.9)
- added R8: 300, Resistor_SMD:R_0603_1608Metric_Pad1.05x0.95mm_HandSolder, F.Cu at (104.2, 94.9)
- added U6: LT1677CS8, ltc1677:SO-8_S, B.Cu at (106.4, 90.0)
- moved J1 4.14 mm to (128.0, 115.9), turned to 225 degrees
- moved C2 2.56 mm to (105.7, 85.0)
- moved C1 2.56 mm to (108.6, 85.0)
- moved C3 2.56 mm to (103.6, 85.0)
- moved U5 2.47 mm to (107.0, 85.0)
- moved U3 0.95 mm to (94.6, 120.2)
Connections:
- U1 pad 11: /tsl237_freq -> /dac_v
- U1 pad 27: Net-(U1-Pad27) -> /irange_0
- U1 pad 28: Net-(U1-Pad28) -> /irange_1
- U1 pad 29: Net-(U1-Pad29) -> /irange_2
- U1 pad 30: Net-(U1-Pad30) -> /irange_3
- U1 pad 6: Net-(U1-Pad6) -> /tsl237_freq
Routing:
- net /dac_v: track 0.00 -> 41.8 mm, vias 0 -> 4
- net GND: track 51.3 -> 87.0 mm, vias 7 -> 14
- net /tsl237_pwr: track 35.2 -> 62.4 mm, vias 4 -> 6
- net /irange_3: track 0.00 -> 26.0 mm, vias 0 -> 3
- net /irange_2: track 0.00 -> 25.5 mm, vias 0 -> 5
- net /current_feedback: track 0.00 -> 23.9 mm, vias 0 -> 3
- net /irange_1: track 0.00 -> 20.3 mm, vias 0 -> 3
- net Net-(U1-Pad14): track 18.9 -> 0.00 mm, vias 3 -> 0
- net /irange_0: track 0.00 -> 18.6 mm, vias 0 -> 3
- net Net-(D2-Pad2): track 0.00 -> 16.6 mm, vias 0 -> 1
- net /sensor_3v: track 29.0 -> 44.2 mm, vias 1 -> 3
- net Net-(J1-Pad2): track 23.3 -> 31.4 mm, vias 0 -> 3
- net Net-(J1-Pad1): track 25.5 -> 33.5 mm, vias 0 -> 3
- net Net-(D1-Pad2): track 4.16 -> 0.00 mm
- net Net-(IC1-Pad3): track 26.0 -> 30.1 mm, vias 0 -> 4
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Other:
- board text added: "Dark Sky Detector R009"
- board text removed: "Dark Sky Detector R008"

Commit message: rev 10 board
Parts:
- removed H2: MountingHole, MountingHole:MountingHole_2.2mm_M2_Pad_Via
- added C4: 0.1uF, Capacitor_SMD:C_0603_1608Metric_Pad1.05x0.95mm_HandSolder, F.Cu at (103.9, 110.4)
- added C5: 1uF, Capacitor_SMD:C_0603_1608Metric_Pad1.05x0.95mm_HandSolder, F.Cu at (120.0, 86.2)
- added C6: 0.1uF, Capacitor_SMD:C_0603_1608Metric_Pad1.05x0.95mm_HandSolder, F.Cu at (121.6, 86.2)
- added C7: 0.1uF, Capacitor_SMD:C_0603_1608Metric_Pad1.05x0.95mm_HandSolder, F.Cu at (107.9, 109.5)
- added G***: LOGO, logo:iu_trident, F.Cu at (121.0, 98.6)
- added G***: LOGO, logo:hnf_logo, F.Cu at (131.8, 98.5)
- added R1: R_US, Resistor_SMD:R_0603_1608Metric_Pad1.05x0.95mm_HandSolder, B.Cu at (97.6, 117.4)
- added R10: R_US, Resistor_SMD:R_0603_1608Metric_Pad1.05x0.95mm_HandSolder, F.Cu at (116.8, 85.4)
- added R11: R_US, Resistor_SMD:R_0603_1608Metric_Pad1.05x0.95mm_HandSolder, F.Cu at (107.9, 112.8)
- added R12: R_US, Resistor_SMD:R_0603_1608Metric_Pad1.05x0.95mm_HandSolder, F.Cu at (111.4, 112.8)
- added R9: R_US, Resistor_SMD:R_0603_1608Metric_Pad1.05x0.95mm_HandSolder, F.Cu at (97.6, 117.4)
- added TP1: TestPoint, TestPoint:TestPoint_Pad_D1.5mm, F.Cu at (127.5, 87.3)
- added TP10: TestPoint, TestPoint:TestPoint_Pad_D1.5mm, F.Cu at (117.5, 109.3)
- added TP11: TestPoint, TestPoint:TestPoint_Pad_D1.5mm, F.Cu at (91.0, 112.3)
- added TP2: TestPoint, TestPoint:TestPoint_Pad_D1.5mm, F.Cu at (102.9, 107.1)
- added TP3: TestPoint, TestPoint:TestPoint_Pad_D1.5mm, F.Cu at (97.2, 122.1)
- added TP4: TestPoint, TestPoint:TestPoint_Pad_D1.5mm, F.Cu at (121.4, 89.8)
- added TP5: TestPoint, TestPoint:TestPoint_Pad_D1.5mm, F.Cu at (109.0, 114.9)
- added TP6: TestPoint, TestPoint:TestPoint_Pad_D1.5mm, F.Cu at (108.4, 90.1)
- added TP7: TestPoint, TestPoint:TestPoint_Pad_D1.5mm, F.Cu at (111.7, 115.9)
- added TP8: TestPoint, TestPoint:TestPoint_Pad_D1.5mm, F.Cu at (109.4, 101.9)
- added TP9: TestPoint, TestPoint:TestPoint_Pad_D1.5mm, F.Cu at (108.5, 95.0)
- BT1: footprint bhimebau_battery:BR2330A_Horizontal_Circular_Holes -> bhimebau_battery:TLH-5935
- C1, C2: value 2.2uF -> 1uF
- C3: value 0.1uF -> 1uF; moved to F.Cu
- R3, R4: moved to F.Cu
- U4: value sm_tsl237 -> TPS7A05; footprint bhimebau_lightsensor:tsl237t -> Package_TO_SOT_SMD:SOT-23; moved to B.Cu
- U5: value REG710-3 -> TPS22917
- U6: value LT1677CS8 -> AD8515; footprint ltc1677:SO-8_S -> Package_TO_SOT_SMD:SOT-353_SC-70-5_Handsoldering; moved to F.Cu
- moved J1 23.3 mm to (104.9, 119.1), turned to 270 degrees
- moved U6 19.8 mm to (110.1, 109.5), turned to 90 degrees
- moved U4 19.1 mm to (124.3, 86.0)
- moved C2 17.7 mm to (123.4, 86.1)
- moved J2 17.5 mm to (107.1, 84.6), turned to 207 degrees
- moved C1 16.4 mm to (125.0, 86.2)
- moved R2 16.4 mm to (105.8, 92.2), turned to 90 degrees
- moved JP1 16.1 mm to (120.0, 83.0), turned to 180 degrees
- moved C3 14.8 mm to (118.4, 86.2)
- moved U5 13.2 mm to (120.0, 86.2)
- moved U3 12.8 mm to (105.7, 113.9), turned to 0 degrees
- moved R7 11.1 mm to (110.2, 105.1), turned to 90 degrees
- moved R8 11.1 mm to (108.5, 105.1), turned to 90 degrees
- moved R5 10.9 mm to (105.1, 105.1), turned to 90 degrees
- moved R6 10.2 mm to (106.8, 105.1), turned to 90 degrees
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Connections:
- net /tsl237_pwr renamed /sensor_pwr
- C1 pad 1: /sensor_3v -> +BATT
- C3 pad 1: Net-(C3-Pad1) -> +BATT
- C3 pad 2: Net-(C3-Pad2) -> GND
- D2 pad 1: /current_feedback -> Net-(D2-Pad1)
- IC1 pad 2: /sensor_3v -> +VSW
- JP1 pad 2: VDD -> +BATT
- R5 pad 1: /current_feedback -> Net-(D2-Pad1)
- R6 pad 1: /current_feedback -> Net-(D2-Pad1)
- R7 pad 1: /current_feedback -> Net-(D2-Pad1)
- R8 pad 1: /current_feedback -> Net-(D2-Pad1)
- U1 pad 12: Net-(U1-Pad12) -> /batt_measure
- U1 pad 18: Net-(U1-Pad18) -> /CLKOUT
- U4 pad 2: GND -> VDD
- U4 pad 3: /sensor_3v -> +BATT
- U5 pad 1: /sensor_3v -> +BATT
- U5 pad 4: Net-(C3-Pad2) -> Net-(C5-Pad1)
- U5 pad 5: VDD -> Net-(R10-Pad1)
- U5 pad 6: Net-(C3-Pad1) -> +VSW
- U6 pad 1: Net-(U6-Pad1) -> Net-(D2-Pad2)
- U6 pad 2: /current_feedback -> GND
- U6 pad 3: /dac_v -> Net-(R11-Pad1)
- U6 pad 4: GND -> Net-(D2-Pad1)
- U6 pad 5: Net-(U6-Pad5) -> +VSW
Routing:
- net +VSW: track 0.00 -> 55.1 mm, vias 0 -> 5
- net VDD: track 17.8 -> 67.0 mm, vias 5 -> 8
- net /sensor_3v: track 44.2 -> 0.00 mm, vias 3 -> 0
- net GND: track 87.0 -> 46.4 mm, vias 14 -> 7
- net Net-(J1-Pad1): track 33.5 -> 2.12 mm, vias 3 -> 0
- net Net-(J1-Pad2): track 31.4 -> 2.20 mm, vias 3 -> 0
- net /dac_v: track 41.8 -> 14.4 mm, vias 4 -> 1
- net /TX: track 47.2 -> 21.8 mm, vias 5 -> 2
- net Net-(BT1-Pad1): track 6.00 -> 31.3 mm, vias 0 -> 1
- net /current_feedback: track 23.9 -> 0.00 mm, vias 3 -> 0
- net Net-(IC1-Pad3): track 30.1 -> 7.12 mm, vias 4 -> 0
- net /RX: track 53.6 -> 33.3 mm
- net /irange_3: track 26.0 -> 9.88 mm, vias 3 -> 1
- net +BATT: track 0.00 -> 15.1 mm, vias 0 -> 2
- net Net-(D2-Pad1): track 0.00 -> 13.8 mm
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Other:
- board text added: "Dark Sky Detector R010"
- board text removed: "Dark Sky Detector R009"

Commit message: save off before access from freecad
Parts:
- added D1: LED, LED_SMD:LED_0603_1608Metric_Pad1.05x0.95mm_HandSolder, F.Cu at (113.5, 97.0)
- added R13: 4.7k, Resistor_SMD:R_0603_1608Metric_Pad1.05x0.95mm_HandSolder, F.Cu at (113.5, 98.7)
- C10: value 2.2uF -> 1uF
- C5: value 1uF -> 680pf
- C7: value 0.1uF -> 1uF
- R1: renamed from R9; value R_US -> 10k
- R5: value 47k -> 46.4k
- R8: value 300 -> 316
- R9: renamed from R1; value R_US -> 10k
- moved D2 2.85 mm to (113.5, 105.0)
- moved G*** 0.75 mm to (121.8, 98.3)
- moved G*** 0.65 mm to (131.5, 99.1)
Routing:
- net Net-(R13-Pad1): track 0.00 -> 49.7 mm, vias 0 -> 1
- net Net-(D2-Pad2): track 12.9 -> 15.7 mm
- net Net-(D2-Pad1): track 13.8 -> 16.1 mm
- net Net-(D1-Pad2): track 0.00 -> 1.70 mm
- net GND: track 46.4 -> 47.6 mm, vias 7 -> 8
Other:
- board text added: "Dark Sky Detector R011"
- board text removed: "Dark Sky Detector R010"

Commit message: added all changed files
Parts:
- removed G***: LOGO, logo:iu_trident
- removed G***: LOGO, logo:hnf_logo
- J1: footprint Connector_JST:JST_XH_B3B-XH-AM_1x03_P2.50mm_Vertical -> Connector_JST:JST_XH_B3B-XH-A_1x03_P2.50mm_Vertical
- J2: footprint Connector_JST:JST_XH_B4B-XH-AM_1x04_P2.50mm_Vertical -> Connector_JST:JST_XH_B4B-XH-A_1x04_P2.50mm_Vertical
- R11, R12: value R_US -> 100k
- U1: footprint Housings_DFN_QFN:QFN-32-1EP_5x5mm_Pitch0.5mm -> Package_DFN_QFN:QFN-32-1EP_5x5mm_P0.5mm_EP3.6x3.6mm
